Commit message: ddpg

File: rbt_description/urdf/fetch.urdf (robot description, URDF)
Before this commit: robot rbt, 3 links, 2 joints
Links:
- added link bellows_link, mass 0.169374038216602; collision mesh filename=package://fetch_description/meshes/bellows_link_collision.S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; visual mesh filename=package://fetch_description/meshes/bellows_link.STL
- added link bellows_link2, mass 0.169374038216602; collision mesh filename=package://fetch_description/meshes/bellows_link_collision.S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; visual mesh filename=package://fetch_description/meshes/bellows_link.STL
- added link elbow_flex_link, mass 2.1299; collision mesh filename=package://fetch_description/meshes/elbow_flex_link_collisio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; visual mesh filename=package://fetch_description/meshes/elbow_flex_link.dae
- added link estop_link, mass 0.00196130439134723; collision mesh filename=package://fetch_description/meshes/estop_link.STL; visual mesh filename=package://fetch_description/meshes/estop_link.STL
- added link forearm_roll_link, mass 1.6563; collision mesh filename=package://fetch_description/meshes/forearm_roll_link_collis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; visual mesh filename=package://fetch_description/meshes/forearm_roll_link.dae
- added link gripper_link, mass 1.5175; collision mesh filename=package://fetch_description/meshes/gripper_link.STL; visual mesh filename=package://fetch_description/meshes/gripper_link.dae
- added link head_camera_depth_frame
- added link head_camera_depth_optical_frame
- added link head_camera_link
- added link head_camera_rgb_frame
- added link head_camera_rgb_optical_frame
- added link head_pan_link, mass 2.2556; collision mesh filename=package://fetch_description/meshes/head_pan_link_collision.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; visual mesh filename=package://fetch_description/meshes/head_pan_link.dae
- added link head_tilt_link, mass 0.9087; collision mesh filename=package://fetch_description/meshes/head_tilt_link_collision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; visual mesh filename=package://fetch_description/meshes/head_tilt_link.dae
- added link l_gripper_finger_link, mass 0.0798; collision mesh filename=package://fetch_description/meshes/l_gripper_finger_link.STL; visual mesh filename=package://fetch_description/meshes/l_gripper_finger_link.STL
- added link laser_link, mass 0.00833634573995571; collision mesh filename=package://fetch_description/meshes/laser_link.STL; visual mesh filename=package://fetch_description/meshes/laser_link.STL
- added link r_gripper_finger_link, mass 0.0798; collision mesh filename=package://fetch_description/meshes/r_gripper_finger_link.STL; visual mesh filename=package://fetch_description/meshes/r_gripper_finger_link.STL
- added link shoulder_lift_link, mass 2.6615; collision mesh filename=package://fetch_description/meshes/shoulder_lift_link_colli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; visual mesh filename=package://fetch_description/meshes/shoulder_lift_link.dae
- added link shoulder_pan_link, mass 2.5587; collision mesh filename=package://fetch_description/meshes/shoulder_pan_link_collis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; visual mesh filename=package://fetch_description/meshes/shoulder_pan_link.dae
- added link torso_fixed_link, mass 13.2775; collision mesh filename=package://fetch_description/meshes/torso_fixed_link.STL; visual mesh filename=package://fetch_description/meshes/torso_fixed_link.dae
- added link torso_lift_link, mass 10.7796; collision mesh filename=package://fetch_description/meshes/torso_lift_link_collisio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; visual mesh filename=package://fetch_description/meshes/torso_lift_link.dae
- added link upperarm_roll_link, mass 2.3311; collision mesh filename=package://fetch_description/meshes/upperarm_roll_link_colli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; visual mesh filename=package://fetch_description/meshes/upperarm_roll_link.dae
- added link wrist_flex_link, mass 1.725; collision mesh filename=package://fetch_description/meshes/wrist_flex_link_collisio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; visual mesh filename=package://fetch_description/meshes/wrist_flex_link.dae
- added link wrist_roll_link, mass 0.1354; collision mesh filename=package://fetch_description/meshes/wrist_roll_link_collisio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; visual mesh filename=package://fetch_description/meshes/wrist_roll_link.dae
- link base_link: geometry collision mesh filename=package://fetch_description/meshes/base_link_collision.STL; visual mesh filename=package://fetch_description/meshes/base_link.dae
- link l_wheel_link: geometry collision mesh filename=package://fetch_description/meshes/l_wheel_link_collision.S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; visual mesh filename=package://fetch_description/meshes/l_wheel_link.STL
- link r_wheel_link: geometry collision mesh filename=package://fetch_description/meshes/r_wheel_link_collision.S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; visual mesh filename=package://fetch_description/meshes/r_wheel_link.STL
Joints:
- added joint bellows_joint: type prismatic, parent torso_lift_link, child bellows_link, origin xyz=0 0 0 rpy=0 0 0, axis 0 0 -1, limit lower=0 upper=0.4 effort=5.0 velocity=0.1
- added joint bellows_joint2: type fixed, parent torso_lift_link, child bellows_link2, origin xyz=0 0 0 rpy=0 0 0
- added joint elbow_flex_joint: type revolute, parent upperarm_roll_link, child elbow_flex_link, origin xyz=0.133 0 0 rpy=0 0 0, axis 0 1 0, limit lower=-2.251 upper=2.251 effort=66.18 velocity=1.521
- added joint estop_joint: type fixed, parent base_link, child estop_link, origin xyz=-0.12465 0.23892 0.31127 rpy=1.5708 0 0, axis 0 0 0
- added joint forearm_roll_joint: type continuous, parent elbow_flex_link, child forearm_roll_link, origin xyz=0.197 0 0 rpy=0 0 0, axis 1 0 0, limit effort=29.35 velocity=1.571
- added joint gripper_axis: type fixed, parent wrist_roll_link, child gripper_link, origin xyz=0.16645 0 0 rpy=0 0 0, axis 0 1 0
- added joint head_camera_depth_joint: type fixed, parent head_camera_link, child head_camera_depth_frame, origin xyz=0 0.045 0 rpy=0 0 0
- added joint head_camera_depth_optical_joint: type fixed, parent head_camera_depth_frame, child head_camera_depth_optical_frame, origin xyz=0 0 0 rpy=-1.57079632679 0 -1.57079632679
- added joint head_camera_joint: type fixed, parent head_tilt_link, child head_camera_link, origin xyz=0.055 0 0.0225 rpy=0 0 0
- added joint head_camera_rgb_joint: type fixed, parent head_camera_link, child head_camera_rgb_frame, origin xyz=0 0.02 0 rpy=0 0 0
- added joint head_camera_rgb_optical_joint: type fixed, parent head_camera_rgb_frame, child head_camera_rgb_optical_frame, origin xyz=0 0 0 rpy=-1.57079632679 0 -1.57079632679
- added joint head_pan_joint: type revolute, parent torso_lift_link, child head_pan_link, origin xyz=0.053125 0 0.603001417713939 rpy=0 0 0, axis 0 0 1, limit lower=-1.57 upper=1.57 effort=0.32 velocity=1.57
- added joint head_tilt_joint: type revolute, parent head_pan_link, child head_tilt_link, origin xyz=0.14253 0 0.057999 rpy=0 0 0, axis 0 1 0, limit lower=-0.76 upper=1.45 effort=0.68 velocity=1.57
- added joint l_gripper_finger_joint: type prismatic, parent gripper_link, child l_gripper_finger_link, origin xyz=0 -0.015425 0 rpy=0 0 0, axis 0 -1 0, limit lower=0.0 upper=0.05 effort=60 velocity=0.05
- added joint laser_joint: type fixed, parent base_link, child laser_link, origin xyz=0.235 0 0.2878 rpy=3.14159265359 0 0, axis 0 0 0
- added joint r_gripper_finger_joint: type prismatic, parent gripper_link, child r_gripper_finger_link, origin xyz=0 0.015425 0 rpy=0 0 0, axis 0 1 0, limit lower=0.0 upper=0.05 effort=60 velocity=0.05
- added joint shoulder_lift_joint: type revolute, parent shoulder_pan_link, child shoulder_lift_link, origin xyz=0.117 0 0.0599999999999999 rpy=0 0 0, axis 0 1 0, limit lower=-1.221 upper=1.518 effort=131.76 velocity=1.454
- added joint shoulder_pan_joint: type revolute, parent torso_lift_link, child shoulder_pan_link, origin xyz=0.119525 0 0.34858 rpy=0 0 0, axis 0 0 1, limit lower=-1.6056 upper=1.6056 effort=33.82 velocity=1.256
- added joint torso_fixed_joint: type fixed, parent base_link, child torso_fixed_link, origin xyz=-0.086875 0 0.377425 rpy=-6.12303176911189E-17 0 0, axis 0 1 0
- added joint torso_lift_joint: type prismatic, parent base_link, child torso_lift_link, origin xyz=-0.086875 0 0.37743 rpy=-6.123E-17 0 0, axis 0 0 1, limit lower=0 upper=0.38615 effort=450.0 velocity=0.1
- added joint upperarm_roll_joint: type continuous, parent shoulder_lift_link, child upperarm_roll_link, origin xyz=0.219 0 0 rpy=0 0 0, axis 1 0 0, limit effort=76.94 velocity=1.571
- added joint wrist_flex_joint: type revolute, parent forearm_roll_link, child wrist_flex_link, origin xyz=0.1245 0 0 rpy=0 0 0, axis 0 1 0, limit lower=-2.16 upper=2.16 effort=25.7 velocity=2.268
- added joint wrist_roll_joint: type continuous, parent wrist_flex_link, child wrist_roll_link, origin xyz=0.1385 0 0 rpy=0 0 0, axis 1 0 0, limit effort=7.36 velocity=2.268

File: rbt_description/urdf/rbt.xacro (robot description, xacro)
@@ -2,19 +2,19 @@
 <robot name="rbt" xmlns:xacro="http://www.ros.org/wiki/xacro">
  <xacro:include filename="$(find rbt_gazebo)/robots/rbt.gazebo.xacro" />
- <link
+   <link
     name="base_link">
     <inertial>
       <origin
-        xyz="0.0015246 0.1254 -0.017729"
-        rpy="0 0 0" />
-      <mass
-        value="70" />
-      <inertia
-        ixx="1.225"
-        ixy="0.0099"
-        ixz="0.0062"
-        iyy="1.2853"
-        iyz="-0.0034"
-        izz="0.987" />
+        xyz="0.0010903 0.26955 -0.073337"
+        rpy="0 0 0" />
+      <mass
+        value="613.17" />
+      <inertia
+        ixx="0"
+        ixy="0"
+        ixz="0"
+        iyy="0"
+        iyz="0"
+        izz="0" />
     </inertial>
     <visual>
@@ -42,19 +42,72 @@
     </collision>
   </link>
+  <link
+    name="r_wheel_link">
+    <inertial>
+      <origin
+        xyz="-2.5535E-15 -4.8572E-17 -0.015"
+        rpy="0 0 0" />
+      <mass
+        value="0.14401" />
+      <inertia
+        ixx="0"
+        ixy="0"
+        ixz="0"
+        iyy="0"
+        iyz="0"
+        izz="0" />
+    </inertial>
+    <visual>
+      <origin
+        xyz="0 0 0"
+        rpy="0 0 0" />
+      <geometry>
+        <mesh
+          filename="package://rbt_description/meshes/r_wheel_link.STL" />
+      </geometry>
+      <material
+        name="">
+        <color
+          rgba="0.0078431 0 0.027451 1" />
+      </material>
+    </visual>
+    <collision>
+      <origin
+        xyz="0 0 0"
+        rpy="0 0 0" />
+      <geometry>
+        <mesh
+          filename="package://rbt_description/meshes/r_wheel_link.STL" />
+      </geometry>
+    </collision>
+  </link>
+  <joint
+    name="r_wheel_joint"
+    type="continuous">
+    <origin
+      xyz="-0.175 0.1 0.05"
+      rpy="1.5708 6.123E-17 1.5708" />
+    <parent
+      link="base_link" />
+    <child
+      link="r_wheel_link" />
+    <axis
+      xyz="0 0 1" />
+  </joint>
   <link
     name="l_wheel_link">
     <inertial>
       <origin
-        xyz="6.8001E-16 3.4694E-18 0.19"
-        rpy="0 0 0" />
-      <mass
-        value="4.3542" />
-      <inertia
-        ixx="0.0045"
-        ixy="0"
-        ixz="0"
-        iyy="0.005"
-        iyz="0"
-        izz="0.0045" />
+        xyz="0.09 0.05 0.19"
+        rpy="0 0 0" />
+      <mass
+        value="0.14401" />
+      <inertia
+        ixx="0"
+        ixy="0"
+        ixz="0"
+        iyy="0"
+        iyz="0"
+        izz="0" />
     </inertial>
     <visual>
@@ -86,5 +139,5 @@
     type="continuous">
     <origin
-      xyz="0 0.1 0.025"
+      xyz="0 0.01 0"
       rpy="1.5708 6.123E-17 1.5708" />
     <parent
@@ -94,63 +147,62 @@
     <axis
       xyz="0 0 1" />
-    <limit
-      effort="8.85"
-      velocity="17.4" />
   </joint>
   <link
-    name="r_wheel_link">
-    <inertial>
-      <origin
-        xyz="-1.2351E-15 0 -0.025524"
-        rpy="0 0 0" />
-      <mass
-        value="0.14401" />
-      <inertia
-        ixx="0.0045"
-        ixy="0"
-        ixz="0"
-        iyy="0.005"
-        iyz="0"
-        izz="0.0045" />
-    </inertial>
-    <visual>
-      <origin
-        xyz="0 0 0"
-        rpy="0 0 0" />
-      <geometry>
-        <mesh
-          filename="package://rbt_description/meshes/r_wheel_link.STL" />
-      </geometry>
-      <material
-        name="">
-        <color
-          rgba="0.0078431 0 0.027451 1" />
-      </material>
-    </visual>
-    <collision>
-      <origin
-        xyz="0 0 0"
-        rpy="0 0 0" />
-      <geometry>
-        <mesh
-          filename="package://rbt_description/meshes/r_wheel_link.STL" />
+    name="shoulder_link">
+    <inertial>
+      <origin
+        xyz="-3.4958E-06 0.014067 0.0085834"
+        rpy="0 0 0" />
+      <mass
+        value="0.30688" />
+      <inertia
+        ixx="0"
+        ixy="0"
+        ixz="0"
+        iyy="0"
+        iyz="0"
+        izz="0" />
+    </inertial>
+    <visual>
+      <origin
+        xyz="0 0 0"
+        rpy="0 0 0" />
+      <geometry>
+        <mesh
+          filename="package://rbt_description/meshes/shoulder_link.STL" />
+      </geometry>
+      <material
+        name="">
+        <color
+          rgba="0.52941 0.54902 0.54902 1" />
+      </material>
+    </visual>
+    <collision>
+      <origin
+        xyz="0 0 0"
+        rpy="0 0 0" />
+      <geometry>
+        <mesh
+          filename="package://rbt_description/meshes/shoulder_link.STL" />
       </geometry>
     </collision>
   </link>
   <joint
-    name="r_wheel_joint"
-    type="continuous">
+    name="shoulder_joint"
+    type="revolute">
     <origin
-      xyz="-0.16448 0.1 0.025"
-      rpy="1.5708 6.123E-17 1.5708" />
+      xyz="0 0.11378 0.675"
+      rpy="1.5708 0 0" />
     <parent
       link="base_link" />
     <child
-      link="r_wheel_link" />
+      link="shoulder_link" />
     <axis
-      xyz="0 0 1" />
+      xyz="0 1 0" />
     <limit
-      effort="8.85"
-      velocity="17.4" />
+      lower="0"
+      upper="1.57"
+      effort="1"
+      velocity="8" />
   </joint>
 </robot>

File: rbt_gazebo/robots/rbt.gazebo.xacro (robot description, xacro)
@@ -40,4 +40,7 @@
     <implicitSpringDamper>1</implicitSpringDamper>
   </gazebo>
+  <gazebo reference=" shoulder_joint">
+    <implicitSpringDamper>1</implicitSpringDamper>
+  </gazebo>
   <gazebo>
     <plugin name="differential_drive_controller" filename="libgazebo_ros_diff_drive.so">
