Commit message: urdf

File: rbt_description/urdf/rbt.xacro (robot description, xacro)
@@ -1,20 +1,13 @@
-<robot
-  name="rbt_description">
-  <link name="base_footprint">
-    <visual>
-      <origin rpy="0 0 0" xyz="0 0 0"/>
-      <geometry>
-        <box size="0.05 0.05 0.001"/>
-      </geometry>
-    </visual>
-  </link>
+<?xml version="1.0"?>
+<robot name="rbt" xmlns:xacro="http://www.ros.org/wiki/xacro">
+ <xacro:include filename="$(find rbt_gazebo)/robots/rbt.gazebo.xacro" />
   <link
     name="base_link">
     <inertial>
       <origin
-        xyz="0.00101738010389675 0.274716843808839 -0.0788251259866206"
+        xyz="-0.0015246 0.1504 0.017729"
         rpy="0 0 0" />
       <mass
-        value="67.4974297376225" />
+        value="439.78" />
       <inertia
         ixx="0"
@@ -36,5 +29,5 @@
         name="">
         <color
-          rgba="1 1 1 1" />
+          rgba="0.52941 0.54902 0.54902 1" />
       </material>
     </visual>
@@ -49,24 +42,19 @@
     </collision>
   </link>
-  <joint name="base_joint" type="fixed">
-    <origin rpy="0 0 0" xyz="0 0 0"/>
-    <parent link="base_footprint"/>
-    <child link="base_link"/>
-  </joint>
   <link
     name="r_wheel_link">
     <inertial>
       <origin
-        xyz="-0.0125 -9.7145E-17 0"
+        xyz="6.9389E-18 9.7145E-17 -0.015"
         rpy="0 0 0" />
       <mass
-        value="0.14346" />
+        value="0.14401" />
       <inertia
-        ixx="3.1851E-35"
-        ixy="4.3235E-35"
-        ixz="3.7109E-35"
-        iyy="1.1543E-34"
-        iyz="-1.5741E-35"
-        izz="1.2026E-34" />
+        ixx="0"
+        ixy="0"
+        ixz="0"
+        iyy="0"
+        iyz="0"
+        izz="0" />
     </inertial>
     <visual>
@@ -81,5 +69,5 @@
         name="">
         <color
-          rgba="0.75294 0.75294 0.75294 1" />
+          rgba="0.0078431 0 0.027451 1" />
       </material>
     </visual>
@@ -98,6 +86,6 @@
     type="continuous">
     <origin
-      xyz="-0.178 0.098 0.0666"
-      rpy="0 0 0" />
+      xyz="0.175 -0.1 0.05"
+      rpy="1.5708 1.4293 -1.5708" />
     <parent
       link="base_link" />
@@ -105,5 +93,5 @@
       link="r_wheel_link" />
     <axis
-      xyz="1 0 0" />
+      xyz="0 0 -1" />
   </joint>
   <link
@@ -111,15 +99,15 @@
     <inertial>
       <origin
-        xyz="0.0125 1.8874E-15 4.996E-16"
+        xyz="6.9389E-18 9.7145E-17 0.015"
         rpy="0 0 0" />
       <mass
-        value="0.14346" />
+        value="0.14401" />
       <inertia
-        ixx="6.3702E-36"
-        ixy="1.2358E-35"
-        ixz="3.0982E-36"
-        iyy="1.1089E-34"
-        iyz="-1.5026E-36"
-        izz="1.1651E-34" />
+        ixx="0"
+        ixy="0"
+        ixz="0"
+        iyy="0"
+        iyz="0"
+        izz="0" />
     </inertial>
     <visual>
@@ -134,5 +122,5 @@
         name="">
         <color
-          rgba="0.75294 0.75294 0.75294 1" />
+          rgba="0.0078431 0 0.027451 1" />
       </material>
     </visual>
@@ -151,6 +139,6 @@
     type="continuous">
     <origin
-      xyz="0.178 0.098 0.0666"
-      rpy="0 0 0" />
+      xyz="-0.175 -0.1 0.05"
+      rpy="1.5708 1.4293 -1.5708" />
     <parent
       link="base_link" />
@@ -158,5 +146,5 @@
       link="l_wheel_link" />
     <axis
-      xyz="1 0 0" />
+      xyz="0 0 -1" />
   </joint>
 </robot>

File: rbt_gazebo/robots/rbt.gazebo.xacro (robot description, xacro)
@@ -1,4 +1,3 @@
 <robot xmlns:xacro="http://www.ros.org/wiki/xacro" name= "rbt" >
-  <xacro:include filename="$(find rbt_description)/urdf/rbt.urdf" />
   <!-- Base is modeled as a big tub sitting on floor, with two wheels -->
   <gazebo reference="base_link">

Commit message: freight

File: rbt_description/urdf/rbt.xacro (robot description, xacro)
@@ -2,19 +2,19 @@
 <robot name="rbt" xmlns:xacro="http://www.ros.org/wiki/xacro">
  <xacro:include filename="$(find rbt_gazebo)/robots/rbt.gazebo.xacro" />
-  <link
+ <link
     name="base_link">
     <inertial>
       <origin
-        xyz="-0.0015246 0.1504 0.017729"
+        xyz="0.0015246 0.1254 -0.017729"
         rpy="0 0 0" />
       <mass
-        value="439.78" />
+        value="70" />
       <inertia
-        ixx="0"
-        ixy="0"
-        ixz="0"
-        iyy="0"
-        iyz="0"
-        izz="0" />
+        ixx="1.225"
+        ixy="0.0099"
+        ixz="0.0062"
+        iyy="1.2853"
+        iyz="-0.0034"
+        izz="0.987" />
     </inertial>
     <visual>
@@ -43,18 +43,74 @@
   </link>
   <link
+    name="l_wheel_link">
+    <inertial>
+      <origin
+        xyz="6.8001E-16 3.4694E-18 0.19"
+        rpy="0 0 0" />
+      <mass
+        value="4.3542" />
+      <inertia
+        ixx="0.0045"
+        ixy="0"
+        ixz="0"
+        iyy="0.005"
+        iyz="0"
+        izz="0.0045" />
+    </inertial>
+    <visual>
+      <origin
+        xyz="0 0 0"
+        rpy="0 0 0" />
+      <geometry>
+        <mesh
+          filename="package://rbt_description/meshes/l_wheel_link.STL" />
+      </geometry>
+      <material
+        name="">
+        <color
+          rgba="0.0078431 0 0.027451 1" />
+      </material>
+    </visual>
+    <collision>
+      <origin
+        xyz="0 0 0"
+        rpy="0 0 0" />
+      <geometry>
+        <mesh
+          filename="package://rbt_description/meshes/l_wheel_link.STL" />
+      </geometry>
+    </collision>
+  </link>
+  <joint
+    name="l_wheel_joint"
+    type="continuous">
+    <origin
+      xyz="0 0.1 0.025"
+      rpy="1.5708 6.123E-17 1.5708" />
+    <parent
+      link="base_link" />
+    <child
+      link="l_wheel_link" />
+    <axis
+      xyz="0 0 1" />
+    <limit
+      effort="8.85"
+      velocity="17.4" />
+  </joint>
+  <link
     name="r_wheel_link">
     <inertial>
       <origin
-        xyz="6.9389E-18 9.7145E-17 -0.015"
+        xyz="-1.2351E-15 0 -0.025524"
         rpy="0 0 0" />
       <mass
         value="0.14401" />
       <inertia
-        ixx="0"
+        ixx="0.0045"
         ixy="0"
         ixz="0"
-        iyy="0"
+        iyy="0.005"
         iyz="0"
-        izz="0" />
+        izz="0.0045" />
     </inertial>
     <visual>
@@ -86,6 +142,6 @@
     type="continuous">
     <origin
-      xyz="0.175 -0.1 0.05"
-      rpy="1.5708 1.4293 -1.5708" />
+      xyz="-0.16448 0.1 0.025"
+      rpy="1.5708 6.123E-17 1.5708" />
     <parent
       link="base_link" />
@@ -93,58 +149,8 @@
       link="r_wheel_link" />
     <axis
-      xyz="0 0 -1" />
-  </joint>
-  <link
-    name="l_wheel_link">
-    <inertial>
-      <origin
-        xyz="6.9389E-18 9.7145E-17 0.015"
-        rpy="0 0 0" />
-      <mass
-        value="0.14401" />
-      <inertia
-        ixx="0"
-        ixy="0"
-        ixz="0"
-        iyy="0"
-        iyz="0"
-        izz="0" />
-    </inertial>
-    <visual>
-      <origin
-        xyz="0 0 0"
-        rpy="0 0 0" />
-      <geometry>
-        <mesh
-          filename="package://rbt_description/meshes/l_wheel_link.STL" />
-      </geometry>
-      <material
-        name="">
-        <color
-          rgba="0.0078431 0 0.027451 1" />
-      </material>
-    </visual>
-    <collision>
-      <origin
-        xyz="0 0 0"
-        rpy="0 0 0" />
-      <geometry>
-        <mesh
-          filename="package://rbt_description/meshes/l_wheel_link.STL" />
-      </geometry>
-    </collision>
-  </link>
-  <joint
-    name="l_wheel_joint"
-    type="continuous">
-    <origin
-      xyz="-0.175 -0.1 0.05"
-      rpy="1.5708 1.4293 -1.5708" />
-    <parent
-      link="base_link" />
-    <child
-      link="l_wheel_link" />
-    <axis
-      xyz="0 0 -1" />
+      xyz="0 0 1" />
+    <limit
+      effort="8.85"
+      velocity="17.4" />
   </joint>
 </robot>

Commit message: n

File: rbt_description/urdf/rbt.xacro (robot description, xacro)
@@ -2,19 +2,14 @@
 <robot name="rbt" xmlns:xacro="http://www.ros.org/wiki/xacro">
  <xacro:include filename="$(find rbt_gazebo)/robots/rbt.gazebo.xacro" />
-   <link
+  <link
     name="base_link">
     <inertial>
       <origin
-        xyz="0.0010903 0.26955 -0.073337"
+        xyz="1.61180778117708E-17 0.105338647334788 -3.58247598962808E-05"
         rpy="0 0 0" />
       <mass
-        value="613.17" />
+        value="70.1294" />
       <inertia
-        ixx="0"
-        ixy="0"
-        ixz="0"
-        iyy="0"
-        iyz="0"
-        izz="0" />
+        ixx="1.225" ixy="0.0099" ixz="0.0062" iyy="1.2853" iyz="-0.0034" izz="0.987" />
     </inertial>
     <visual>
@@ -27,7 +22,7 @@
       </geometry>
       <material
-        name="">
+        name="Black">
         <color
-          rgba="0.52941 0.54902 0.54902 1" />
+          rgba="0.3 0.3 0.3 1.0" />
       </material>
     </visual>
@@ -43,18 +38,61 @@
   </link>
   <link
+    name="l_wheel_link">
+    <inertial>
+      <origin
+        xyz="3.5354E-16 6.9389E-18 0.015"
+        rpy="0 0 0" />
+      <mass
+        value="4.3542" />
+      <inertia
+       ixx="0.0045" ixy="0" ixz="0" iyy="0.005" iyz="0" izz="0.0045"  />
+    </inertial>
+    <visual>
+      <origin
+        xyz="0 0 0"
+        rpy="0 0 0" />
+      <geometry>
+        <mesh
+          filename="package://rbt_description/meshes/l_wheel_link.STL" />
+      </geometry>
+      <material
+        name="">
+        <color
+          rgba="0 0.17255 1 1" />
+      </material>
+    </visual>
+    <collision>
+      <origin
+        xyz="0 0 0"
+        rpy="0 0 0" />
+      <geometry>
+        <mesh
+          filename="package://rbt_description/meshes/l_wheel_link.STL" />
+      </geometry>
+    </collision>
+  </link>
+  <joint
+    name="l_wheel_joint"
+    type="continuous">
+    <origin
+      xyz="0.165 0 0.05"
+      rpy="1.5708 6.123E-17 1.5708" />
+    <parent
+      link="base_link" />
+    <child
+      link="l_wheel_link" />
+    <axis
+      xyz="0 0 1" />
+  </joint>
+  <link
     name="r_wheel_link">
     <inertial>
       <origin
-        xyz="-2.5535E-15 -4.8572E-17 -0.015"
+        xyz="-9.0369E-16 6.9389E-18 -0.015"
         rpy="0 0 0" />
       <mass
-        value="0.14401" />
+        value="4.3542" />
       <inertia
-        ixx="0"
-        ixy="0"
-        ixz="0"
-        iyy="0"
-        iyz="0"
-        izz="0" />
+        ixx="0.0045" ixy="0" ixz="0" iyy="0.005" iyz="0" izz="0.0045" />
     </inertial>
     <visual>
@@ -69,5 +107,5 @@
         name="">
         <color
-          rgba="0.0078431 0 0.027451 1" />
+          rgba="0 0.17255 1 1" />
       </material>
     </visual>
@@ -86,5 +124,5 @@
     type="continuous">
     <origin
-      xyz="-0.175 0.1 0.05"
+      xyz="-0.165 0 0.05"
       rpy="1.5708 6.123E-17 1.5708" />
     <parent
@@ -96,11 +134,11 @@
   </joint>
   <link
-    name="l_wheel_link">
+    name="laser_link">
     <inertial>
       <origin
-        xyz="0.09 0.05 0.19"
+        xyz="3.2198E-17 -0.0042085 0"
         rpy="0 0 0" />
       <mass
-        value="0.14401" />
+        value="4.3542" />
       <inertia
         ixx="0"
@@ -117,10 +155,10 @@
       <geometry>
         <mesh
-          filename="package://rbt_description/meshes/l_wheel_link.STL" />
+          filename="package://rbt_description/meshes/laser_link.STL" />
       </geometry>
       <material
         name="">
         <color
-          rgba="0.0078431 0 0.027451 1" />
+          rgba="0.79216 0.81961 0.93333 1" />
       </material>
     </visual>
@@ -131,78 +169,20 @@
       <geometry>
         <mesh
-          filename="package://rbt_description/meshes/l_wheel_link.STL" />
+          filename="package://rbt_description/meshes/laser_link.STL" />
       </geometry>
     </collision>
   </link>
   <joint
-    name="l_wheel_joint"
-    type="continuous">
+    name="laser_joint"
+    type="fixed">
     <origin
-      xyz="0 0.01 0"
-      rpy="1.5708 6.123E-17 1.5708" />
-    <parent
-      link="base_link" />
-    <child
-      link="l_wheel_link" />
-    <axis
-      xyz="0 0 1" />
-  </joint>
-  <link
-    name="shoulder_link">
-    <inertial>
-      <origin
-        xyz="-3.4958E-06 0.014067 0.0085834"
-        rpy="0 0 0" />
-      <mass
-        value="0.30688" />
-      <inertia
-        ixx="0"
-        ixy="0"
-        ixz="0"
-        iyy="0"
-        iyz="0"
-        izz="0" />
-    </inertial>
-    <visual>
-      <origin
-        xyz="0 0 0"
-        rpy="0 0 0" />
-      <geometry>
-        <mesh
-          filename="package://rbt_description/meshes/shoulder_link.STL" />
-      </geometry>
-      <material
-        name="">
-        <color
-          rgba="0.52941 0.54902 0.54902 1" />
-      </material>
-    </visual>
-    <collision>
-      <origin
-        xyz="0 0 0"
-        rpy="0 0 0" />
-      <geometry>
-        <mesh
-          filename="package://rbt_description/meshes/shoulder_link.STL" />
-      </geometry>
-    </collision>
-  </link>
-  <joint
-    name="shoulder_joint"
-    type="revolute">
-    <origin
-      xyz="0 0.11378 0.675"
+      xyz="0 -0.21 0.212"
       rpy="1.5708 0 0" />
     <parent
       link="base_link" />
     <child
-      link="shoulder_link" />
+      link="laser_link" />
     <axis
-      xyz="0 1 0" />
-    <limit
-      lower="0"
-      upper="1.57"
-      effort="1"
-      velocity="8" />
+      xyz="0 0 0" />
   </joint>
 </robot>

File: rbt_gazebo/robots/rbt.gazebo.xacro (robot description, xacro)
@@ -2,44 +2,46 @@
   <!-- Base is modeled as a big tub sitting on floor, with two wheels -->
   <gazebo reference="base_link">
-    <kp>100000000.0</kp>
-    <kd>10.0</kd>
-    <mu1>0.1</mu1>
-    <mu2>0.1</mu2>
-    <fdir1>1 0 0</fdir1>
-    <maxVel>10.0</maxVel>
-    <minDepth>0.0005</minDepth>
-    <material>Gazebo/White</material>
+    <material>Gazebo/Black</material>
     <turnGravityOff>false</turnGravityOff>
   </gazebo>
   <gazebo reference="r_wheel_link">
-    <kp>500000.0</kp>
-    <kd>10.0</kd>
-    <mu1>10</mu1>
-    <mu2>10</mu2>
-    <fdir1>1 0 0</fdir1>
-    <maxVel>1.0</maxVel>
-    <minDepth>0.003</minDepth>
-    <material>Gazebo/Black</material>
+    <material>Gazebo/Blue</material>
     <turnGravityOff>false</turnGravityOff>
   </gazebo>
   <gazebo reference="l_wheel_link">
-    <kp>500000.0</kp>
-    <kd>10.0</kd>
-    <mu1>10</mu1>
-    <mu2>10</mu2>
-    <fdir1>1 0 0</fdir1>
-    <maxVel>1.0</maxVel>
-    <minDepth>0.003</minDepth>
-    <material>Gazebo/Black</material>
+    <material>Gazebo/Blue</material>
     <turnGravityOff>false</turnGravityOff>
   </gazebo>
-  <gazebo reference="l_wheel_joint">
-    <implicitSpringDamper>1</implicitSpringDamper>
-  </gazebo>
-  <gazebo reference="r_wheel_joint">
-    <implicitSpringDamper>1</implicitSpringDamper>
-  </gazebo>
-  <gazebo reference=" shoulder_joint">
-    <implicitSpringDamper>1</implicitSpringDamper>
+  <gazebo reference="laser_link">
+    <sensor type="ray" name="laser_link">
+      <pose>0 0 0 0 0 0</pose>
+      <visualize>false</visualize>
+      <update_rate>15</update_rate>
+      <ray>
+        <scan>
+          <horizontal>
+            <samples>662</samples>
+            <resolution>1</resolution>
+            <min_angle>-1.91986</min_angle>
+            <max_angle>1.91986</max_angle>
+          </horizontal>
+        </scan>
+        <range>
+          <min>0.05</min>
+          <max>25.0</max>
+          <resolution>0.01</resolution>
+        </range>
+        <noise>
+          <!-- Noise parameters based on spec for SICK TIM561 (10m version) -->
+          <type>gaussian</type>
+          <mean>0.0</mean>
+          <stddev>0.02</stddev>
+        </noise>
+      </ray>
+      <plugin name="gazebo_ros_base_hokuyo_controller" filename="libgazebo_ros_laser.so">
+        <topicName>/scan</topicName>
+        <frameName>laser_link</frameName>
+      </plugin>
+    </sensor>
   </gazebo>
   <gazebo>
@@ -61,5 +63,5 @@
       <commandTopic>cmd_vel</commandTopic>
       <odometryFrame>odom</odometryFrame>
-      <odometryTopic>odom</odometryTopic>
+      <odometryTopic>/odom</odometryTopic>
       <robotBaseFrame>base_link</robotBaseFrame>
     </plugin>

Commit message: gaz

File: rbt_description/urdf/rbt.xacro (robot description, xacro)
@@ -6,10 +6,15 @@
     <inertial>
       <origin
-        xyz="1.61180778117708E-17 0.105338647334788 -3.58247598962808E-05"
+        xyz="1.5170507548791E-17 -0.000197277236774495 0.0803276867224908"
         rpy="0 0 0" />
       <mass
-        value="70.1294" />
+        value="190.047063870531" />
       <inertia
-        ixx="1.225" ixy="0.0099" ixz="0.0062" iyy="1.2853" iyz="-0.0034" izz="0.987" />
+        ixx="0.00513222256327552"
+        ixy="1.43114686768087E-17"
+        ixz="3.46944695195361E-18"
+        iyy="0.0118016516978085"
+        iyz="-0.00113704440589145"
+        izz="0.0164025460146906" />
     </inertial>
     <visual>
@@ -22,7 +27,7 @@
       </geometry>
       <material
-        name="Black">
+        name="">
         <color
-          rgba="0.3 0.3 0.3 1.0" />
+          rgba="0.752941176470588 0.752941176470588 0.752941176470588 1" />
       </material>
     </visual>
@@ -41,10 +46,15 @@
     <inertial>
       <origin
-        xyz="3.5354E-16 6.9389E-18 0.015"
+        xyz="0 0 0.015"
         rpy="0 0 0" />
       <mass
-        value="4.3542" />
+        value="0.144199844682647" />
       <inertia
-       ixx="0.0045" ixy="0" ixz="0" iyy="0.005" iyz="0" izz="0.0045"  />
+        ixx="0"
+        ixy="0"
+        ixz="0"
+        iyy="0"
+        iyz="0"
+        izz="0" />
     </inertial>
     <visual>
@@ -59,5 +69,5 @@
         name="">
         <color
-          rgba="0 0.17255 1 1" />
+          rgba="1 1 1 1" />
       </material>
     </visual>
@@ -76,6 +86,6 @@
     type="continuous">
     <origin
-      xyz="0.165 0 0.05"
-      rpy="1.5708 6.123E-17 1.5708" />
+      xyz="0.185 0.13 0.05"
+      rpy="1.5707963267949 6.12303176911189E-17 1.5707963267949" />
     <parent
       link="base_link" />
@@ -89,10 +99,15 @@
     <inertial>
       <origin
-        xyz="-9.0369E-16 6.9389E-18 -0.015"
+        xyz="-5.55111512312578E-17 6.93889390390723E-18 -0.015"
         rpy="0 0 0" />
       <mass
-        value="4.3542" />
+        value="0.144199844682647" />
       <inertia
-        ixx="0.0045" ixy="0" ixz="0" iyy="0.005" iyz="0" izz="0.0045" />
+        ixx="0"
+        ixy="0"
+        ixz="0"
+        iyy="0"
+        iyz="0"
+        izz="0" />
     </inertial>
     <visual>
@@ -107,5 +122,5 @@
         name="">
         <color
-          rgba="0 0.17255 1 1" />
+          rgba="1 1 1 1" />
       </material>
     </visual>
@@ -124,6 +139,6 @@
     type="continuous">
     <origin
-      xyz="-0.165 0 0.05"
-      rpy="1.5708 6.123E-17 1.5708" />
+      xyz="-0.185 0.129999999999999 0.0500000000000007"
+      rpy="1.5707963267949 6.12303176911189E-17 1.5707963267949" />
     <parent
       link="base_link" />
@@ -133,56 +148,3 @@
       xyz="0 0 1" />
   </joint>
-  <link
-    name="laser_link">
-    <inertial>
-      <origin
-        xyz="3.2198E-17 -0.0042085 0"
-        rpy="0 0 0" />
-      <mass
-        value="4.3542" />
-      <inertia
-        ixx="0"
-        ixy="0"
-        ixz="0"
-        iyy="0"
-        iyz="0"
-        izz="0" />
-    </inertial>
-    <visual>
-      <origin
-        xyz="0 0 0"
-        rpy="0 0 0" />
-      <geometry>
-        <mesh
-          filename="package://rbt_description/meshes/laser_link.STL" />
-      </geometry>
-      <material
-        name="">
-        <color
-          rgba="0.79216 0.81961 0.93333 1" />
-      </material>
-    </visual>
-    <collision>
-      <origin
-        xyz="0 0 0"
-        rpy="0 0 0" />
-      <geometry>
-        <mesh
-          filename="package://rbt_description/meshes/laser_link.STL" />
-      </geometry>
-    </collision>
-  </link>
-  <joint
-    name="laser_joint"
-    type="fixed">
-    <origin
-      xyz="0 -0.21 0.212"
-      rpy="1.5708 0 0" />
-    <parent
-      link="base_link" />
-    <child
-      link="laser_link" />
-    <axis
-      xyz="0 0 0" />
-  </joint>
 </robot>

File: rbt_gazebo/robots/rbt.gazebo.xacro (robot description, xacro)
@@ -2,46 +2,14 @@
   <!-- Base is modeled as a big tub sitting on floor, with two wheels -->
   <gazebo reference="base_link">
-    <material>Gazebo/Black</material>
+    <material>Gazebo/White</material>
     <turnGravityOff>false</turnGravityOff>
   </gazebo>
   <gazebo reference="r_wheel_link">
-    <material>Gazebo/Blue</material>
+    <material>Gazebo/White</material>
     <turnGravityOff>false</turnGravityOff>
   </gazebo>
   <gazebo reference="l_wheel_link">
-    <material>Gazebo/Blue</material>
+    <material>Gazebo/White</material>
     <turnGravityOff>false</turnGravityOff>
-  </gazebo>
-  <gazebo reference="laser_link">
-    <sensor type="ray" name="laser_link">
-      <pose>0 0 0 0 0 0</pose>
-      <visualize>false</visualize>
-      <update_rate>15</update_rate>
-      <ray>
-        <scan>
-          <horizontal>
-            <samples>662</samples>
-            <resolution>1</resolution>
-            <min_angle>-1.91986</min_angle>
-            <max_angle>1.91986</max_angle>
-          </horizontal>
-        </scan>
-        <range>
-          <min>0.05</min>
-          <max>25.0</max>
-          <resolution>0.01</resolution>
-        </range>
-        <noise>
-          <!-- Noise parameters based on spec for SICK TIM561 (10m version) -->
-          <type>gaussian</type>
-          <mean>0.0</mean>
-          <stddev>0.02</stddev>
-        </noise>
-      </ray>
-      <plugin name="gazebo_ros_base_hokuyo_controller" filename="libgazebo_ros_laser.so">
-        <topicName>/scan</topicName>
-        <frameName>laser_link</frameName>
-      </plugin>
-    </sensor>
   </gazebo>
   <gazebo>
@@ -56,6 +24,6 @@
       <leftJoint>l_wheel_joint</leftJoint>
       <rightJoint>r_wheel_joint</rightJoint>
-      <wheelSeparation>300</wheelSeparation>
-      <wheelDiameter>80</wheelDiameter>
+      <wheelSeparation>400</wheelSeparation>
+      <wheelDiameter>100</wheelDiameter>
       <broadcastTF>1</broadcastTF>
       <wheelTorque>30</wheelTorque>
@@ -63,5 +31,5 @@
       <commandTopic>cmd_vel</commandTopic>
       <odometryFrame>odom</odometryFrame>
-      <odometryTopic>/odom</odometryTopic>
+      <odometryTopic>odom</odometryTopic>
       <robotBaseFrame>base_link</robotBaseFrame>
     </plugin>
