Commit message: urdf

File: rbt_description/urdf/rbt.urdf (robot description, URDF)
Before this commit: robot rbt_description, 3 links, 2 joints
Links:
- added link base_footprint; visual box size=0.05 0.05 0.001
- link base_link: mass 66.903 -> 67.4974297376225
Joints:
- added joint base_joint: type fixed, parent base_footprint, child base_link, origin xyz=0 0 0 rpy=0 0 0
- joint l_wheel_joint: origin xyz=0.178 -0.152 0.0806 rpy=-0.24564 0 0 -> xyz=0.178 0.098 0.0666 rpy=0 0 0
- joint r_wheel_joint: axis 0 0 1 -> 1 0 0; origin xyz=-0.178 -0.152 0.0806 rpy=1.5708 -1.5378 1.5708 -> xyz=-0.178 0.098 0.0666 rpy=0 0 0

Commit message: gaz

File: rbt_description/urdf/rbt.urdf (robot description, URDF)
Before this commit: robot rbt, 3 links, 2 joints
Links:
- link base_link: mass 190.047063870531 -> 70.1294
- link l_wheel_link: mass 0.144199844682647 -> 4.3542
- link r_wheel_link: mass 0.144199844682647 -> 4.3542

File: rbt_gazebo/robots/rbt.gazebo.xacro (robot description, xacro)
@@ -1,15 +1,39 @@
 <robot xmlns:xacro="http://www.ros.org/wiki/xacro" name= "rbt" >
+  <xacro:include filename="$(find rbt_description)/urdf/rbt.urdf" />
   <!-- Base is modeled as a big tub sitting on floor, with two wheels -->
   <gazebo reference="base_link">
-    <material>Gazebo/White</material>
-    <turnGravityOff>false</turnGravityOff>
+    <kp>100000000.0</kp>
+    <kd>10.0</kd>
+    <mu1>0.1</mu1>
+    <mu2>0.1</mu2>
+    <fdir1>1 0 0</fdir1>
+    <maxVel>10.0</maxVel>
+    <minDepth>0.0005</minDepth>
   </gazebo>
   <gazebo reference="r_wheel_link">
-    <material>Gazebo/White</material>
-    <turnGravityOff>false</turnGravityOff>
+    <kp>500000.0</kp>
+    <kd>10.0</kd>
+    <mu1>10</mu1>
+    <mu2>10</mu2>
+    <fdir1>1 0 0</fdir1>
+    <maxVel>1.0</maxVel>
+    <minDepth>0.003</minDepth>
+    <material>Gazebo/Blue</material>
   </gazebo>
   <gazebo reference="l_wheel_link">
-    <material>Gazebo/White</material>
-    <turnGravityOff>false</turnGravityOff>
+    <kp>500000.0</kp>
+    <kd>10.0</kd>
+    <mu1>10</mu1>
+    <mu2>10</mu2>
+    <fdir1>1 0 0</fdir1>
+    <maxVel>1.0</maxVel>
+    <minDepth>0.003</minDepth>
+    <material>Gazebo/Blue</material>
+  </gazebo>
+<gazebo reference="l_wheel_joint">
+    <implicitSpringDamper>1</implicitSpringDamper>
+  </gazebo>
+  <gazebo reference="r_wheel_joint">
+    <implicitSpringDamper>1</implicitSpringDamper>
   </gazebo>
   <gazebo>

Commit message: tens
ddpg_tens

File: rbt_description/urdf/rbt.urdf (robot description, URDF)
Before this commit: robot rbt, 3 links, 2 joints
Links:
- link r_wheel_link: geometry collision mesh filename=package://rbt_description/meshes/r_wheel_link.dae; visual mesh filename=package://rbt_description/meshes/r_wheel_link.dae

Commit message: s1

File: rbt_description/urdf/rbt.urdf (robot description, URDF)
Before this commit: robot rbt, 3 links, 2 joints
Links:
- added link laser_link, mass 0.11769; collision mesh filename=package://rbt_description/meshes/laser_link.STL; visual mesh filename=package://rbt_description/meshes/laser_link.STL
- link base_link: mass 70.1294 -> 34.8310964963823
- link l_wheel_link: mass 4.3542 -> 0.38838
- link r_wheel_link: mass 4.3542 -> 0.38838; geometry collision mesh filename=package://rbt_description/meshes/r_wheel_link.STL; visual mesh filename=package://rbt_description/meshes/r_wheel_link.STL
Joints:
- added joint laser_joint: type fixed, parent base_link, child laser_link, origin xyz=0.165 0 0.257 rpy=1.5777E-30 -2.3314E-29 -3.2868E-15, axis 0 0 0
- joint l_wheel_joint: axis 0 0 1 -> 0 -1 0; origin xyz=0.185 0.13 0.05 rpy=1.5707963267949 6.12303176911189E-17 1.5707963267949 -> xyz=-0.12 0.175 0.07 rpy=1.5777E-30 -2.3314E-29 -3.2868E-15
- joint r_wheel_joint: axis 0 0 1 -> 0 -1 0; origin xyz=-0.185 0.129999999999999 0.0500000000000007 rpy=1.5707963267949 6.12303176911189E-17 1.5707963267949 -> xyz=-0.12 -0.175 0.07 rpy=1.5777E-30 -2.3314E-29 -3.2868E-15

Commit message: s1

File: rbt_description/urdf/rbt.urdf (robot description, URDF)
Before this commit: robot rbt, 4 links, 3 joints
Links:
- link base_link: geometry collision mesh filename=package://rbt_description/meshes/base_link.STL; visual mesh filename=package://rbt_description/meshes/base_link.dae
- link l_wheel_link: geometry collision mesh filename=package://rbt_description/meshes/l_wheel_link.STL; visual mesh filename=package://rbt_description/meshes/l_wheel_link.dae
- link laser_link: geometry collision mesh filename=package://rbt_description/meshes/laser_link.STL; visual mesh filename=package://rbt_description/meshes/laser_link.dae
- link r_wheel_link: geometry collision mesh filename=package://rbt_description/meshes/r_wheel_link.STL; visual mesh filename=package://rbt_description/meshes/r_wheel_link.dae

Commit message: s2

File: rbt_description/urdf/rbt.urdf (robot description, URDF)
Before this commit: robot rbt, 4 links, 3 joints
Links:
- link l_wheel_link: mass 0.38838 -> 3.8838
- link r_wheel_link: mass 0.38838 -> 3.8838
Joints:
- joint l_wheel_joint: axis 0 -1 0 -> 0 1 0
- joint r_wheel_joint: axis 0 -1 0 -> 0 1 0

File: rbt_gazebo/robots/rbt.gazebo.xacro (robot description, xacro)
@@ -59,3 +59,35 @@
     </plugin>
   </gazebo>
+  <gazebo reference="laser_link">
+    <sensor type="ray" name="base_laser">
+      <pose>0 0 0 0 0 0</pose>
+      <visualize>false</visualize>
+      <update_rate>15</update_rate>
+      <ray>
+        <scan>
+          <horizontal>
+            <samples>662</samples>
+            <resolution>1</resolution>
+            <min_angle>-1.91986</min_angle>
+            <max_angle>1.91986</max_angle>
+          </horizontal>
+        </scan>
+        <range>
+          <min>0.05</min>
+          <max>25.0</max>
+          <resolution>0.01</resolution>
+        </range>
+        <noise>
+          <!-- Noise parameters based on spec for SICK TIM561 (10m version) -->
+          <type>gaussian</type>
+          <mean>0.0</mean>
+          <stddev>0.02</stddev>
+        </noise>
+      </ray>
+      <plugin name="gazebo_ros_base_hokuyo_controller" filename="libgazebo_ros_laser.so">
+        <topicName>/scan</topicName>
+        <frameName>laser_link</frameName>
+      </plugin>
+    </sensor>
+  </gazebo>
 </robot>

Commit message: s3

File: rbt_description/urdf/rbt.urdf (robot description, URDF)
Before this commit: robot rbt, 4 links, 3 joints
Links:
- added link elbow_flex_link, mass 2.1299; collision mesh filename=package://rbt_description/meshes/elbow_flex_link.STL; visual mesh filename=package://rbt_description/meshes/elbow_flex_link.STL
- added link forearm_roll_link, mass 1.6563; collision mesh filename=package://rbt_description/meshes/forearm_roll_link.STL; visual mesh filename=package://rbt_description/meshes/forearm_roll_link.STL
- added link gripper_link, mass 1.5175; collision mesh filename=package://rbt_description/meshes/gripper_link.STL; visual mesh filename=package://rbt_description/meshes/gripper_link.STL
- added link l_gripper_link, mass 0.0798; collision mesh filename=package://rbt_description/meshes/l_gripper_link.STL; visual mesh filename=package://rbt_description/meshes/l_gripper_link.STL
- added link r_gripper_link, mass 0.0798; collision mesh filename=package://rbt_description/meshes/r_gripper_link.STL; visual mesh filename=package://rbt_description/meshes/r_gripper_link.STL
- added link shoulder_lift_link, mass 2.6615; collision mesh filename=package://rbt_description/meshes/shoulder_lift_link.STL; visual mesh filename=package://rbt_description/meshes/shoulder_lift_link.STL
- added link shoulder_pan_link, mass 2.5587; collision mesh filename=package://rbt_description/meshes/shoulder_pan_link.STL; visual mesh filename=package://rbt_description/meshes/shoulder_pan_link.STL
- added link torso_link, mass 13.2775; collision mesh filename=package://rbt_description/meshes/torso_link.STL; visual mesh filename=package://rbt_description/meshes/torso_link.STL
- added link upperarm_roll_link, mass 2.3311; collision mesh filename=package://rbt_description/meshes/upperarm_roll_link.STL; visual mesh filename=package://rbt_description/meshes/upperarm_roll_link.STL
- added link wrist_flex_link, mass 1.725; collision mesh filename=package://rbt_description/meshes/wrist_flex_link.STL; visual mesh filename=package://rbt_description/meshes/wrist_flex_link.STL
- added link wrist_roll_link, mass 0.1354; collision mesh filename=package://rbt_description/meshes/wrist_roll_link.STL; visual mesh filename=package://rbt_description/meshes/wrist_roll_link.STL
Joints:
- added joint elbow_flex_joint: type revolute, parent upperarm_roll_link, child elbow_flex_link, origin xyz=0.10000000000001 0.000172781781224759 0.0012087169179047 rpy=-3.54831426125384E-43 -1.01364733915118E-30 0, axis 0 1 0, limit lower=-2.251 upper=2.251 effort=66.18 velocity=1.521
- added joint forearm_roll_joint: type continuous, parent elbow_flex_link, child forearm_roll_link, origin xyz=0.1 0 0 rpy=-3.47545734981105E-43 0 0, axis 1 0 0, limit effort=29.35 velocity=1.571
- added joint gripper_joint: type fixed, parent wrist_roll_link, child gripper_link, origin xyz=0.02 0 0 rpy=-3.4755E-43 0 0, axis 0 0 0
- added joint l_gripper_joint: type prismatic, parent gripper_link, child l_gripper_link, origin xyz=0.0199999999999914 0.0114999999999914 0 rpy=-3.47545734981105E-43 0 0, axis 0 -1 0, limit lower=-0.005 upper=0.01 effort=60 velocity=0.05
- added joint r_gripper_joint: type prismatic, parent gripper_link, child r_gripper_link, origin xyz=0.0199999999999908 -0.0114999999999821 0 rpy=-3.47545734981105E-43 0 0, axis 0 1 0, limit lower=-0.005 upper=0.01 effort=60 velocity=0.05
- added joint shoulder_lift_joint: type revolute, parent shoulder_pan_link, child shoulder_lift_link, origin xyz=0.139999999999999 0.0275000000000008 0.0799999999999998 rpy=-3.47545734981105E-43 0 0, axis 0 1 0, limit lower=-1.221 upper=1.518 effort=131.76 velocity=1.454
- added joint shoulder_pan_joint: type revolute, parent torso_link, child shoulder_pan_link, origin xyz=0.16 0 0.545 rpy=-3.54831426125384E-43 -1.01364733915118E-30 0, axis 0 0 1, limit lower=-1.6056 upper=1.6056 effort=33.82 velocity=1.256
- added joint torso_joint: type fixed, parent base_link, child torso_link, origin xyz=-0.19 0 0.225 rpy=-3.47545734981105E-43 1.01364733915118E-30 0, axis 0 0 0
- added joint upperarm_roll_joint: type continuous, parent shoulder_lift_link, child upperarm_roll_link, origin xyz=0.100000000000014 0 0 rpy=-3.47545734981105E-43 1.01364733915118E-30 0, axis 1 0 0, limit effort=76.94 velocity=1.571
- added joint wrist_flex_joint: type revolute, parent forearm_roll_link, child wrist_flex_link, origin xyz=0.126633249580691 -0.00252269168014944 0 rpy=-3.47545734981105E-43 0 0, axis 0 1 0, limit lower=-2.16 upper=2.16 effort=25.7 velocity=2.268
- added joint wrist_roll_joint: type continuous, parent wrist_flex_link, child wrist_roll_link, origin xyz=0.12 0 0 rpy=-3.47545734981105E-43 0 0, axis 1 0 0, limit effort=7.36 velocity=2.268

File: rbt_gazebo/robots/rbt.gazebo.xacro (robot description, xacro)
@@ -36,4 +36,28 @@
   <gazebo reference="r_wheel_joint">
     <implicitSpringDamper>1</implicitSpringDamper>
+  </gazebo>
+  <gazebo reference="forearm_roll_joint">
+    <implicitSpringDamper>1</implicitSpringDamper>
+  </gazebo>
+  <gazebo reference="wrist_roll_joint">
+    <implicitSpringDamper>1</implicitSpringDamper>
+  </gazebo>
+  <gazebo reference="r_gripper_link">
+    <kp>1000000.0</kp>
+    <kd>100.0</kd>
+    <mu1>30.0</mu1>
+    <mu2>30.0</mu2>
+    <maxVel>1.0</maxVel>
+    <minDepth>0.001</minDepth>
+    <material>Gazebo/Grey</material>
+  </gazebo>
+  <gazebo reference="l_gripper_link">
+    <kp>1000000.0</kp>
+    <kd>100.0</kd>
+    <mu1>30.0</mu1>
+    <mu2>30.0</mu2>
+    <maxVel>1.0</maxVel>
+    <minDepth>0.001</minDepth>
+    <material>Gazebo/Grey</material>
   </gazebo>
   <gazebo>

Commit message: adding blender

File: rbt_description/urdf/rbt.urdf (robot description, URDF)
Before this commit: robot rbt, 15 links, 14 joints
Links:
- link elbow_flex_link: geometry collision mesh filename=package://rbt_description/meshes/elbow_flex_link.STL; visual mesh filename=package://rbt_description/meshes/elbow_flex_link.dae
- link forearm_roll_link: geometry collision mesh filename=package://rbt_description/meshes/forearm_roll_link.STL; visual mesh filename=package://rbt_description/meshes/forearm_roll_link.dae
- link gripper_link: geometry collision mesh filename=package://rbt_description/meshes/gripper_link.STL; visual mesh filename=package://rbt_description/meshes/gripper_link.dae
- link l_gripper_link: geometry collision mesh filename=package://rbt_description/meshes/l_gripper_link.STL; visual mesh filename=package://rbt_description/meshes/l_gripper_link.dae
- link r_gripper_link: geometry collision mesh filename=package://rbt_description/meshes/r_gripper_link.STL; visual mesh filename=package://rbt_description/meshes/r_gripper_link.dae
- link shoulder_lift_link: geometry collision mesh filename=package://rbt_description/meshes/shoulder_lift_link.STL; visual mesh filename=package://rbt_description/meshes/shoulder_lift_link.dae
- link shoulder_pan_link: geometry collision mesh filename=package://rbt_description/meshes/shoulder_pan_link.STL; visual mesh filename=package://rbt_description/meshes/shoulder_pan_link.dae
- link torso_link: geometry collision mesh filename=package://rbt_description/meshes/torso_link.STL; visual mesh filename=package://rbt_description/meshes/torso_link.dae
- link upperarm_roll_link: geometry collision mesh filename=package://rbt_description/meshes/upperarm_roll_link.STL; visual mesh filename=package://rbt_description/meshes/upperarm_roll_link.dae
- link wrist_flex_link: geometry collision mesh filename=package://rbt_description/meshes/wrist_flex_link.STL; visual mesh filename=package://rbt_description/meshes/wrist_flex_link.dae
- link wrist_roll_link: geometry collision mesh filename=package://rbt_description/meshes/wrist_roll_link.STL; visual mesh filename=package://rbt_description/meshes/wrist_roll_link.dae

Commit message: v1

File: rbt_description/urdf/rbt.urdf (robot description, URDF)
Before this commit: robot rbt, 15 links, 14 joints
Links:
- removed link elbow_flex_link
- removed link forearm_roll_link
- removed link gripper_link
- removed link l_gripper_link
- removed link r_gripper_link
- removed link upperarm_roll_link
- removed link wrist_flex_link
- removed link wrist_roll_link
- link base_link: mass 34.8310964963823 -> 5.0
Joints:
- removed joint elbow_flex_joint
- removed joint forearm_roll_joint
- removed joint gripper_joint
- removed joint l_gripper_joint
- removed joint r_gripper_joint
- removed joint upperarm_roll_joint
- removed joint wrist_flex_joint
- removed joint wrist_roll_joint

File: rbt_gazebo/robots/rbt.gazebo.xacro (robot description, xacro)
@@ -37,4 +37,5 @@
     <implicitSpringDamper>1</implicitSpringDamper>
   </gazebo>
+<!--
   <gazebo reference="forearm_roll_joint">
     <implicitSpringDamper>1</implicitSpringDamper>
@@ -61,4 +62,5 @@
     <material>Gazebo/Grey</material>
   </gazebo>
+-->
   <gazebo>
     <plugin name="differential_drive_controller" filename="libgazebo_ros_diff_drive.so">
@@ -115,12 +117,13 @@
     </sensor>
   </gazebo>
-<gazebo reference="shoulder_pan_link">
-    <kp>100000000.0</kp>
-    <kd>10.0</kd>
-    <mu1>0.1</mu1>
-    <mu2>0.1</mu2>
-    <fdir1>1 0 0</fdir1>
-    <maxVel>10.0</maxVel>
-    <minDepth>0.0005</minDepth>
+   <gazebo reference="shoulder_lift_link">
+             <kp>5000.0</kp>
+    <kd>1.0</kd>
+    <material>Gazebo/Grey</material>
+  </gazebo>
+   <gazebo reference="shoulder_pan_link">
+      <kp>5000.0</kp>
+       <kd>1.0</kd>
+       <material>Gazebo/Grey</material>
   </gazebo>
 </robot>

Commit message: v2

File: rbt_description/urdf/rbt.urdf (robot description, URDF)
Before this commit: robot rbt, 7 links, 6 joints
Links:
- link base_link: geometry collision mesh filename=package://rbt_description/meshes/modif/base_link.stl; visual mesh filename=package://rbt_description/meshes/modif/base_link.dae
- link l_wheel_link: mass 3.8838 -> 1.5; geometry collision mesh filename=package://rbt_description/meshes/modif/l_wheel_link.STL; visual mesh filename=package://rbt_description/meshes/modif/l_wheel_link.dae
- link laser_link: geometry collision mesh filename=package://rbt_description/meshes/modif/laser_link.STL; visual mesh filename=package://rbt_description/meshes/modif/laser_link.dae
- link r_wheel_link: mass 3.8838 -> 1.5; geometry collision mesh filename=package://rbt_description/meshes/modif/r_wheel_link.STL; visual mesh filename=package://rbt_description/meshes/modif/r_wheel_link.dae
- link shoulder_lift_link: geometry collision mesh filename=package://rbt_description/meshes/modif/shoulder_lift_link.S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; visual mesh filename=package://rbt_description/meshes/modif/shoulder_lift_link.d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
- link shoulder_pan_link: geometry collision mesh filename=package://rbt_description/meshes/modif/shoulder_pan_link.STL; visual mesh filename=package://rbt_description/meshes/modif/shoulder_pan_link.dae
- link torso_link: geometry collision mesh filename=package://rbt_description/meshes/modif/torso_link.STL; visual mesh filename=package://rbt_description/meshes/modif/torso_link.dae

Commit message: rr

File: rbt_description/urdf/rbt.urdf (robot description, URDF)
Before this commit: robot rbt, 7 links, 6 joints
Links:
- added link upperarm_roll_link, mass 2.3311; collision mesh filename=package://rbt_description/meshes/upperarm_roll_link.STL; visual mesh filename=package://rbt_description/meshes/upperarm_roll_link.dae
- link base_link: mass 5.0 -> 15.000; geometry collision mesh filename=package://rbt_description/meshes/base_link.STL; visual mesh filename=package://rbt_description/meshes/base_link.dae
- link l_wheel_link: mass 1.5 -> 3.8838; geometry collision mesh filename=package://rbt_description/meshes/l_wheel_link.STL; visual mesh filename=package://rbt_description/meshes/l_wheel_link.dae
- link laser_link: geometry collision mesh filename=package://rbt_description/meshes/laser_link.STL; visual mesh filename=package://rbt_description/meshes/laser_link.dae
- link r_wheel_link: mass 1.5 -> 3.8838; geometry collision mesh filename=package://rbt_description/meshes/r_wheel_link.STL; visual mesh filename=package://rbt_description/meshes/r_wheel_link.dae
- link shoulder_lift_link: mass 2.6615 -> 2.2; geometry collision mesh filename=package://rbt_description/meshes/shoulder_lift_link.STL; visual mesh filename=package://rbt_description/meshes/shoulder_lift_link.dae
- link shoulder_pan_link: mass 2.5587 -> 2.2; geometry collision mesh filename=package://rbt_description/meshes/shoulder_pan_link.STL; visual mesh filename=package://rbt_description/meshes/shoulder_pan_link.dae
- link torso_link: geometry collision mesh filename=package://rbt_description/meshes/torso_link.STL; visual mesh filename=package://rbt_description/meshes/torso_link.dae
Joints:
- added joint upperarm_roll_joint: type continuous, parent shoulder_lift_link, child upperarm_roll_link, origin xyz=0.100000000000014 0 0 rpy=-3.47545734981105E-43 1.01364733915118E-30 0, axis 1 0 0, limit effort=76.94 velocity=1.571

File: rbt_gazebo/robots/rbt.gazebo.xacro (robot description, xacro)
@@ -117,13 +117,3 @@
     </sensor>
   </gazebo>
-   <gazebo reference="shoulder_lift_link">
-             <kp>5000.0</kp>
-    <kd>1.0</kd>
-    <material>Gazebo/Grey</material>
-  </gazebo>
-   <gazebo reference="shoulder_pan_link">
-      <kp>5000.0</kp>
-       <kd>1.0</kd>
-       <material>Gazebo/Grey</material>
-  </gazebo>
 </robot>

Commit message: g

File: rbt_description/urdf/rbt.urdf (robot description, URDF)
Before this commit: robot rbt, 8 links, 7 joints
Links:
- removed link shoulder_lift_link
- removed link shoulder_pan_link
- removed link torso_link
- removed link upperarm_roll_link
Joints:
- removed joint shoulder_lift_joint
- removed joint shoulder_pan_joint
- removed joint torso_joint
- removed joint upperarm_roll_joint

Commit message: gazebo

File: rbt_description/urdf/rbt.urdf (robot description, URDF)
Before this commit: robot rbt, 4 links, 3 joints
Links:
- link base_link: mass 15.000 -> 70.1294
- link l_wheel_link: mass 3.8838 -> 4.3542
- link r_wheel_link: mass 3.8838 -> 4.3542
Joints:
- joint laser_joint: axis 0 0 0 -> (none)

File: rbt_gazebo/robots/rbt.gazebo.xacro (robot description, xacro)
@@ -1,5 +1,4 @@
 <robot xmlns:xacro="http://www.ros.org/wiki/xacro" name= "rbt" >
   <xacro:include filename="$(find rbt_description)/urdf/rbt.urdf" />
-  <!-- Base is modeled as a big tub sitting on floor, with two wheels -->
   <gazebo reference="base_link">
     <kp>100000000.0</kp>
@@ -33,34 +32,9 @@
 <gazebo reference="l_wheel_joint">
     <implicitSpringDamper>1</implicitSpringDamper>
-  </gazebo>
-  <gazebo reference="r_wheel_joint">
+</gazebo>
+<gazebo reference="r_wheel_joint">
     <implicitSpringDamper>1</implicitSpringDamper>
-  </gazebo>
+</gazebo>
 <!--
-  <gazebo reference="forearm_roll_joint">
-    <implicitSpringDamper>1</implicitSpringDamper>
-  </gazebo>
-  <gazebo reference="wrist_roll_joint">
-    <implicitSpringDamper>1</implicitSpringDamper>
-  </gazebo>
-  <gazebo reference="r_gripper_link">
-    <kp>1000000.0</kp>
-    <kd>100.0</kd>
-    <mu1>30.0</mu1>
-    <mu2>30.0</mu2>
-    <maxVel>1.0</maxVel>
-    <minDepth>0.001</minDepth>
-    <material>Gazebo/Grey</material>
-  </gazebo>
-  <gazebo reference="l_gripper_link">
-    <kp>1000000.0</kp>
-    <kd>100.0</kd>
-    <mu1>30.0</mu1>
-    <mu2>30.0</mu2>
-    <maxVel>1.0</maxVel>
-    <minDepth>0.001</minDepth>
-    <material>Gazebo/Grey</material>
-  </gazebo>
--->
   <gazebo>
     <plugin name="differential_drive_controller" filename="libgazebo_ros_diff_drive.so">
@@ -117,3 +91,4 @@
     </sensor>
   </gazebo>
+-->
 </robot>
